Commit message: change config of simulation LaserScan

File: src/bumperbot_description/urdf/bumperbot.urdf.xacro (robot description, xacro)
@@ -201,5 +201,5 @@
     <parent link="base_link"/>
     <child link="laser_link"/>
-    <origin xyz="0.0 0.0 0.1208" rpy="0 0 3.14"/>
+    <origin xyz="0.0 0.0 0.1208" rpy="0 0 0"/>
   </joint>
   <material name="blue">

Commit message: update config description for LaserScan

File: src/bumperbot_description/urdf/bumperbot.urdf.xacro (robot description, xacro)
@@ -199,7 +199,8 @@
   </link>
   <joint name="laser_joint" type="fixed">
-    <parent link="base_link"/>
-    <child link="laser_link"/>
-    <origin xyz="0.0 0.0 0.1208" rpy="0 0 0"/>
+    <origin xyz="-0.0050526 -0.0023221 0.1208" rpy="0 0 3.14" />
+    <parent link="base_link" />
+    <child link="laser_link" />
+    <axis xyz="0 0 0" />
   </joint>
   <material name="blue">
